File: NOGGIN/NOGGIN.kicad_pcb (KiCad board)
At the start: 2 copper layers, 63 parts, among them J1 CAN, J2 CAN, J3 SWD_UART, J4 Extra, J5 I2C, J6 UART, J7 DAC1, J8 DAC2, J9 MOTOR, SW1 DBG2, SW2 DBG1, SW3 RST, U1 STM32F072CBUx, U2 AZ1117-3.3, U3 ATA6561, U4 MCP6L02x-xMS, U5 INA2181, U6 DRV8871DDA

Commit message: Finished NOGGIN layout
Parts:
- removed C18, C19: 100n, Capacitor_SMD:C_0603_1608Metric
- removed R5, R6: 10k, Resistor_SMD:R_0603_1608Metric
- removed R7, R8: 5m, Resistor_SMD:R_1206_3216Metric
- added  : version_dots, extraparts:version_dots, F.Cu at (139.8, 84.5)
- added G***: LOGO, extraparts:bac_logo, B.Cu at (160.5, 111.8)
- added G***: LOGO, extraparts:auv_logo, B.Cu at (140.0, 86.5)
- C11, C13, C14, C15, C16, C5, C7, C9, F2, R13, R14, R15, R16, R18, R4, U2: moved to B.Cu
- F1: footprint Fuse:Fuse_2920_7451Metric -> Fuse:Fuse_1206_3216Metric; moved to B.Cu
- J4: footprint Connector_PinHeader_1.27mm:PinHeader_2x09_P1.27mm_Vertical -> Connector_PinSocket_1.27mm:PinSocket_2x07_P1.27mm_Vertical_SMD; moved to B.Cu
- U4: value MCP6L02x-xMS -> ACS70331; footprint Package_SO:MSOP-8_3x3mm_P0.65mm -> Sensor_Current:Allegro_QFN-12-10-1EP_3x3mm_P0.5mm
- U5: value INA2181 -> ACS70331; footprint Package_SO:VSSOP-10_3x3mm_P0.5mm -> Sensor_Current:Allegro_QFN-12-10-1EP_3x3mm_P0.5mm
- moved R14 67.2 mm to (139.8, 90.0)
- moved C10 62.4 mm to (155.0, 96.8), turned to 270 degrees
- moved F1 56.6 mm to (165.0, 113.0)
- moved R15 56.0 mm to (150.8, 94.8), turned to 270 degrees
- moved R13 55.8 mm to (139.8, 91.5)
- moved C12 55.4 mm to (146.5, 95.0)
- moved R19 55.3 mm to (148.5, 109.8), turned to 270 degrees
- moved C7 53.6 mm to (153.5, 105.0), turned to 180 degrees
- moved C11 53.1 mm to (146.5, 95.0)
- moved R18 51.7 mm to (148.5, 105.8), turned to 90 degrees
- moved J6 49.3 mm to (149.5, 83.2)
- moved F2 49.1 mm to (165.0, 109.0)
- moved C8 48.9 mm to (153.5, 105.0), turned to 180 degrees
- moved R17 48.1 mm to (148.5, 106.8), turned to 90 degrees
- moved R16 46.5 mm to (152.2, 94.8), turned to 270 degrees
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Connections:
- C17 pad 1: GND -> +3V3
- C17 pad 2: Net-(C17-Pad2) -> GND
- C3 pad 1: /RST -> +3V3
- J4 pad 10: /PB15 -> /PB2
- J4 pad 11: /PB14 -> /PB1
- J4 pad 12: /PB13 -> /PB0
- J4 pad 13: /PB12 -> GND
- J4 pad 14: /PB2 -> GND
- J4 pad 3: /PB9 -> /PA8
- J4 pad 4: /PB8 -> /PB15
- J4 pad 5: /PB5 -> /PB14
- J4 pad 6: /PB4 -> /PB13
- J4 pad 7: /PB3 -> /PB12
- J4 pad 8: /PA15 -> /PB11
- J4 pad 9: /PA8 -> /PB10
- U1 pad 10: /12v_Isens -> /12v_Vsens
- U1 pad 11: /5v_Isens -> /5v_Vsens
- U1 pad 12: /12v_Vsens -> /12v_Isens
- U1 pad 13: /5v_Vsens -> /5v_Isens
- U1 pad 21: /TX -> /PB10
- U1 pad 22: /RX -> /PB11
- U1 pad 38: /PA15 -> /NOGGIN/PA15
- U1 pad 39: /PB3 -> /TX
- U1 pad 40: /PB4 -> /RX
- U1 pad 41: /PB5 -> /NOGGIN/PB5
- U1 pad 45: /PB8 -> /NOGGIN/PB8
- U1 pad 46: /PB9 -> /NOGGIN/PB9
- U4 pad 1: /1v65_1 -> /12v_Sens+
- U4 pad 2: /1v65_1 -> +12V
- U4 pad 3: Net-(C17-Pad2) -> GND
- U4 pad 5: Net-(C17-Pad2) -> Net-(U4-Pad5)
- U4 pad 6: /1v65_2 -> GND
- U4 pad 7: /1v65_2 -> GND
- U4 pad 8: +3V3 -> /12v_Isens
- U5 pad 1: /12v_Isens -> /5v_Sens+
- U5 pad 2: +12V -> +5V
- U5 pad 3: /12v_Sens+ -> GND
- U5 pad 5: /1v65_1 -> Net-(U5-Pad5)
- U5 pad 6: /1v65_2 -> GND
- U5 pad 7: /5v_Sens+ -> GND
- U5 pad 8: +5V -> /5v_Isens
- U5 pad 9: /5v_Isens -> GND
- U6 pad 6: Net-(J9-Pad1) -> Net-(J9-Pad2)
- U6 pad 8: Net-(J9-Pad2) -> Net-(J9-Pad1)
Routing:
- net +5V: track 0.00 -> 48.3 mm, vias 0 -> 2
- net +3V3: track 0.00 -> 43.4 mm, vias 0 -> 10
- net /RST: track 0.00 -> 35.1 mm, vias 0 -> 2
- net /12v_Isens: track 0.00 -> 28.0 mm, vias 0 -> 2
- net +12V: track 0.00 -> 27.3 mm, vias 0 -> 3
- net Net-(F1-Pad2): track 0.00 -> 25.3 mm, vias 0 -> 3
- net /NOGGIN/PA9(UART_TX): track 0.00 -> 24.6 mm
- net /12v_Vsens: track 0.00 -> 23.7 mm, vias 0 -> 2
- net /5v_Isens: track 0.00 -> 22.5 mm, vias 0 -> 2
- net /NOGGIN/SWCLK: track 0.00 -> 21.1 mm
- net /PB12: track 0.00 -> 20.2 mm, vias 0 -> 2
- net /PB10: track 0.00 -> 19.8 mm, vias 0 -> 2
- net /PB14: track 0.00 -> 19.8 mm, vias 0 -> 2
- net /PA8: track 0.00 -> 19.4 mm, vias 0 -> 2
- net /NOGGIN/PA10(UART_RX): track 0.00 -> 19.4 mm
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- added copper zone on In2.Cu, net +3V3
- added copper zone on B.Cu, net GND
- added copper zone on F.Cu, net GND
- added copper zone on In1.Cu, net GND
Other:
- board outline added: 31.2 x 34 mm
- copper layers 2 -> 4
- net class BigPower added: clearance 0.1524, trace_width 0.508, via_dia 0.7112, via_drill 0.4064
- net class Default: clearance 0.1524 -> 0.127; trace_width 0.1524 -> 0.127; via_dia 0.5588 -> 0.4572
- net class SmallPower added: clearance 0.1524, trace_width 0.3048, via_dia 0.508, via_drill 0.254
- rule trace_clearance: 0.1524 -> 0.127
- rule trace_min: 0.1524 -> 0.127
- rule via_min_size: 0.5588 -> 0.4572
- board text added: "NOGGIN v2 by Matthew Tran"
