File: MATE/ESCC/ESCC.kicad_pcb (KiCad board)
At the start: 2 copper layers, 36 x 40 mm, 28 parts, among them J1 Conn_01x03, J2 Conn_01x05, J3 SWD_UART, SW1 RST, SW2 DBG, U1 STM32F072CBUx, U2 AZ1117-3.3, U3 ATA6561, U4 BESC, U5 ACS725xLCTR-30AB

Commit message: convert to kicad 6
Other:
- net class Default removed
