File: templates/noggin_g0b1ke/noggin_g0b1ke.kicad_pcb (KiCad board)
At the start: 2 copper layers, 21 parts, among them J1 CAN, J2 CAN, J3 SWD_UART, SW1 DBG2, SW2 DBG1, SW3 RST, U1 TCAN330G, U2 STM32G0B1KxTxN

Commit message: convert to kicad 6
Other:
- net class Default removed
