File: MATE/PCC/PCC.kicad_pcb (KiCad board)
At the start: 2 copper layers, 23.5 x 44.5 mm, 22 parts, among them J1 Conn_01x03, SW1 SW_DIP_x04, U1 I6A4W020A033V-001-R

Commit message: convert to kicad 6
Other:
- net class Default removed

Commit message: Suphakorn PCC first commit
Parts:
- added H1: MountingHole, MountingHole:MountingHole_3.2mm_M3, F.Cu at (150.1, 79.6)
- J1: footprint extraparts:Samtec_mPOWER_UMPT_RA_3pin -> extraparts:Samtec_mPOWER_UMPS_3pin
- moved R2 2.80 mm to (152.1, 106.5)
- moved R3 2.80 mm to (152.1, 108.0)
- moved R4 2.80 mm to (152.1, 109.5)
- moved R5 2.80 mm to (152.1, 111.0)
- moved SW1 2.80 mm to (146.6, 108.7)
- moved J1 1.00 mm to (150.0, 124.0)
Routing:
- net +48V: track 8.27 -> 12.0 mm, vias 18 -> 40
- net Net-(R2-Pad2): track 7.46 -> 8.67 mm
- net GND: vias 86 -> 66
- net +VSW: vias 26 -> 30
Other:
- board size 23.5 x 44.5 mm -> 23.5 x 51.8 mm

Commit message: Suphakorn PCC2 second commit
Parts:
- moved C2 7.44 mm to (148.8, 97.4), turned to 0 degrees
- moved C1 4.76 mm to (148.8, 94.0), turned to 0 degrees
- moved C5 1.05 mm to (159.3, 91.0)
- moved C4 1.05 mm to (156.1, 91.0)
- moved C3 1.05 mm to (152.8, 91.0)
- moved H1 0.20 mm to (150.1, 79.8)
Routing:
- net GND: vias 66 -> 63
- net +48V: vias 40 -> 39
Other:
- board size 23.5 x 51.8 mm -> 23.5 x 52.5 mm
- board text added: "PCC v2 by Suphakorn"
- board text removed: "PCC v1 by Matthew Tran"

Commit message: PCBv2 third commit
Parts:
- added G***: LOGO, extraparts:auv_logo, F.Cu at (142.3, 79.7)
- J1: footprint extraparts:Samtec_mPOWER_UMPS_3pin -> extraparts:Samtec_mPOWER_UMPT_3pin
- turned J1 to 180 degrees
Routing:
- net GND: vias 63 -> 60
- net +VSW: vias 30 -> 35
- net +48V: vias 39 -> 41
Other:
- board text added: "PCB v2 by Suphakorn"
- board text removed: "PCC v2 by Suphakorn"
