File: MATE/PCC/PCC.kicad_sch (KiCad schematic)
At the start: 22 parts, among them J1 Conn_01x03, SW1 SW_DIP_x04, U1 I6A4W020A033V-001-R

Commit message: Suphakorn PCC first commit
Parts:
- added H1: MountingHole, MountingHole:MountingHole_3.2mm_M3, symbol Mechanical:MountingHole
- J1: footprint extraparts:Samtec_mPOWER_UMPT_RA_3pin -> extraparts:Samtec_mPOWER_UMPS_3pin
Changed lines of the file:
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@@
       (effects (font (size 1.27 1.27)) (justify right))
     )
-    (property "Footprint" "extraparts:Samtec_mPOWER_UMPT_RA_3pin" (id 2) (at 143.51 72.39 0)
+    (property "Footprint" "extraparts:Samtec_mPOWER_UMPS_3pin" (id 2) (at 143.51 72.39 0)
       (effects (font (size 1.27 1.27)) hide)
     )
@@
     (pin "1")
     (pin "2")
+  )
+  (symbol (lib_id "Mechanical:MountingHole") (at 104.14 66.04 0) (unit 1)
+    (in_bom yes) (on_board yes) (fields_autoplaced)
+    (property "Reference" "H1" (id 0) (at 106.68 65.1315 0)
+      (effects (font (size 1.27 1.27)) (justify left))
+    )
+    (property "Value" "MountingHole" (id 1) (at 106.68 67.9066 0)
+      (effects (font (size 1.27 1.27)) (justify left))
+    )
+    (property "Footprint" "MountingHole:MountingHole_3.2mm_M3" (id 2) (at 104.14 66.04 0)
+      (effects (font (size 1.27 1.27)) hide)
+    )
+    (property "Datasheet" "~" (id 3) (at 104.14 66.04 0)
+      (effects (font (size 1.27 1.27)) hide)
+    )
   )
   (sheet_instances
@@
       (reference "D2") (unit 1) (value "LED") (footprint "LED_SMD:LED_0603_1608Metric")
     )
+    (path "/cf1d9385-6ce9-4595-b21b-bdb3d17e619b"
+      (reference "H1") (unit 1) (value "MountingHole") (footprint "MountingHole:MountingHole_3.2mm_M3")
+    )
     (path "/00000000-0000-0000-0000-00006027c37d"
-      (reference "J1") (unit 1) (value "Conn_01x03") (footprint "extraparts:Samtec_mPOWER_UMPT_RA_3pin")
+      (reference "J1") (unit 1) (value "Conn_01x03") (footprint "extraparts:Samtec_mPOWER_UMPS_3pin")
     )
     (path "/00000000-0000-0000-0000-0000602559ec"

Commit message: PCBv2 third commit
Parts:
- J1: footprint extraparts:Samtec_mPOWER_UMPS_3pin -> extraparts:Samtec_mPOWER_UMPT_3pin
Changed lines of the file:
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@@
       (effects (font (size 1.27 1.27)) (justify right))
     )
-    (property "Footprint" "extraparts:Samtec_mPOWER_UMPS_3pin" (id 2) (at 143.51 72.39 0)
+    (property "Footprint" "extraparts:Samtec_mPOWER_UMPT_3pin" (id 2) (at 143.51 72.39 0)
       (effects (font (size 1.27 1.27)) hide)
     )
@@
     )
     (path "/00000000-0000-0000-0000-00006027c37d"
-      (reference "J1") (unit 1) (value "Conn_01x03") (footprint "extraparts:Samtec_mPOWER_UMPS_3pin")
+      (reference "J1") (unit 1) (value "Conn_01x03") (footprint "extraparts:Samtec_mPOWER_UMPT_3pin")
     )
     (path "/00000000-0000-0000-0000-0000602559ec"
