File: General/BMS/BMS.kicad_pcb (KiCad board)
At the start: 2 copper layers, 36 parts, among them J1 CAN, J2 CAN, J3 DuraClik, J4 XT90, J5 XT90, J6 SWD_UART, J7 ExtPwrSw, K1 A3_Relay, Q1 PMV28ENEA, SW2 DBG2, SW3 DBG1, SW4 RST, U1 VXO7803, U2 TCAN330G, U3 STM32G0B1KxTxN, U4 CZ3AG7_HalEfSens

Commit message: Changes: - Working on Layout
Parts:
- Q1: footprint Package_TO_SOT_SMD:SOT-23-5_HandSoldering -> Package_TO_SOT_SMD:SOT-23
- moved J5 207.9 mm to (82.3, 48.9)
- moved C4 195.6 mm to (60.3, 32.4), turned to 90 degrees
- moved C3 188.2 mm to (62.8, 32.4), turned to 90 degrees
- moved U2 183.7 mm to (67.9, 32.4)
- moved C6 170.8 mm to (104.1, 33.0)
- moved C8 170.8 mm to (112.2, 33.0)
- moved C9 170.8 mm to (104.1, 35.5)
- moved C5 170.8 mm to (108.2, 35.5)
- moved C7 170.8 mm to (108.2, 33.0)
- moved Q1 168.9 mm to (58.4, 50.8), turned to -90 degrees
- moved R4 166.6 mm to (66.0, 47.4), turned to 90 degrees
- moved D3 155.7 mm to (20.3, 94.0)
- moved R6 155.7 mm to (26.5, 96.5)
- moved R7 155.7 mm to (30.5, 96.5)
- moved R8 155.7 mm to (30.5, 101.6)
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Routing:
- net Net-(J1-Pad2): track 0.00 -> 22.0 mm
- net /CAN/CANH: track 0.00 -> 21.8 mm
- net Net-(J1-Pad1): track 0.00 -> 21.4 mm
- net /CAN/CANL: track 0.00 -> 21.4 mm
Other:
- board outline added: 72.2 x 72.2 mm

Commit message: Changes:
- Continuing work on layout and added some courtyards to custom footprints
Parts:
- D1, Q1, R3, R4: moved to B.Cu
- moved R8 119.6 mm to (119.4, 21.6), turned to 180 degrees
- moved D3 117.2 mm to (114.9, 24.8)
- moved R6 115.5 mm to (119.4, 27.9), turned to 180 degrees
- moved R7 114.2 mm to (119.4, 24.8), turned to 180 degrees
- moved J6 112.1 mm to (142.9, 34.9)
- moved U3 83.2 mm to (128.3, 35.6)
- moved R1 68.1 mm to (30.2, 48.3)
- moved R2 50.2 mm to (48.9, 85.1)
- moved SW3 23.7 mm to (108.6, 24.8), turned to 180 degrees
- moved U4 20.9 mm to (70.5, 41.5)
- moved D1 19.2 mm to (46.4, 62.2), turned to -90 degrees
- moved SW2 18.9 mm to (108.6, 29.8), turned to 180 degrees
- moved R4 13.8 mm to (61.6, 60.5)
- moved C6 13.7 mm to (117.5, 36.2), turned to -90 degrees
- moved C9 13.6 mm to (117.5, 33.0), turned to 90 degrees
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Connections:
- net Net-(D3-Pad2) renamed /R
- net Net-(D3-Pad3) renamed /G
- net Net-(D3-Pad4) renamed /B
- J7 pad 1: Net-(C1-Pad1) -> +BATT
- J7 pad 2: +BATT -> Net-(C1-Pad1)
Routing:
- net /RST: track 0.00 -> 47.2 mm, vias 0 -> 2
- net +3V3: track 0.00 -> 39.0 mm, vias 0 -> 2
- net /NOGGIN/SWCLK: track 0.00 -> 37.2 mm
- net /NOGGIN/SWDIO: track 0.00 -> 30.5 mm
- net Net-(J1-Pad2): track 22.0 -> 0.00 mm
- net /CAN/CANH: track 21.8 -> 0.00 mm
- net Net-(J1-Pad1): track 21.4 -> 0.00 mm
- net /CAN/CANL: track 21.4 -> 0.00 mm
- net /NOGGIN/RX: track 0.00 -> 19.2 mm
- net /DBG1: track 0.00 -> 17.2 mm
- net /DBG2: track 0.00 -> 14.9 mm
- net /LED_R: track 0.00 -> 12.3 mm
- net /LED_G: track 0.00 -> 10.3 mm
- net /NOGGIN/TX: track 0.00 -> 9.77 mm
- net /LED_B: track 0.00 -> 7.44 mm
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