File: General/BMS/BMS.kicad_sch (KiCad schematic)
At the start: 26 parts, among them J1 CAN, J2 CAN, J3 DuraClik, J4 XT90, J5 XT90, J7 ExtPwrSw, K1 A3_Relay, Q1 PMV28ENEA, SW2 DBG2, SW3 DBG1, SW4 RST, U1 VXO7803, U4 CZ3AG7_HalEfSens

Commit message: Changes:
- Continuing work on layout and added some courtyards to custom footprints
Connections:
- net +BATT: now also J7.1 (Pin_1); no longer J7.2 (Pin_2)
- net R: now reaches D3.2 (RK), R8.2
- net G: now reaches D3.3 (GK), R7.2
- net B: now reaches D3.4 (BK), R6.2
- net at C1.1, U1.1 (IN): now also J7.2 (Pin_2); no longer J7.1 (Pin_1)
Other:
- moved on the sheet: J7
Changed lines of the file:
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@@
   (no_connect (at 121.92 152.4))
   (no_connect (at 121.92 154.94))
-  (no_connect (at 214.63 68.58))
   (no_connect (at 194.31 71.12))
   (no_connect (at 194.31 68.58))
+  (no_connect (at 214.63 68.58))
   (no_connect (at 214.63 71.12))
   (wire (pts (xy 191.77 66.04) (xy 194.31 66.04))
@@
     (effects (font (size 1.27 1.27)) (justify left bottom))
   )
+  (label "B" (at 185.42 143.51 0)
+    (effects (font (size 1.27 1.27)) (justify left bottom))
+  )
   (label "IP" (at 191.77 66.04 0)
     (effects (font (size 1.27 1.27)) (justify left bottom))
@@
   )
   (label "IP" (at 161.29 63.5 0)
+    (effects (font (size 1.27 1.27)) (justify left bottom))
+  )
+  (label "R" (at 185.42 153.67 0)
     (effects (font (size 1.27 1.27)) (justify left bottom))
   )
@@
   )
   (label "MOSFET1" (at 107.95 129.54 0)
+    (effects (font (size 1.27 1.27)) (justify left bottom))
+  )
+  (label "G" (at 185.42 148.59 0)
     (effects (font (size 1.27 1.27)) (justify left bottom))
   )
@@
     (pin "1")
   )
-  (symbol (lib_id "Connector_Generic:Conn_01x02") (at 48.26 128.27 270) (unit 1)
-    (in_bom yes) (on_board yes)
-    (property "Reference" "J7" (id 0) (at 41.91 128.27 90)
-      (effects (font (size 1.27 1.27)) (justify left))
-    )
-    (property "Value" "ExtPwrSw" (id 1) (at 43.18 132.08 90)
-      (effects (font (size 1.27 1.27)) (justify left))
-    )
-    (property "Footprint" "extraparts:Molex_DuraClik_Vert_2pin" (id 2) (at 48.26 128.27 0)
-      (effects (font (size 1.27 1.27)) hide)
-    )
-    (property "Datasheet" "~" (id 3) (at 48.26 128.27 0)
-      (effects (font (size 1.27 1.27)) hide)
-    )
+  (symbol (lib_id "Connector_Generic:Conn_01x02") (at 45.72 128.27 90) (mirror x) (unit 1)
+    (in_bom yes) (on_board yes)
+    (property "Reference" "J7" (id 0) (at 52.07 128.27 90)
+      (effects (font (size 1.27 1.27)) (justify left))
+    )
+    (property "Value" "ExtPwrSw" (id 1) (at 50.8 132.08 90)
+      (effects (font (size 1.27 1.27)) (justify left))
+    )
+    (property "Footprint" "extraparts:Molex_DuraClik_Vert_2pin" (id 2) (at 45.72 128.27 0)
+      (effects (font (size 1.27 1.27)) hide)
+    )
+    (property "Datasheet" "~" (id 3) (at 45.72 128.27 0)
+      (effects (font (size 1.27 1.27)) hide)
+    )
