File: RoboSub/SidePlaneA/NOGGIN_Block.kicad_sch (KiCad schematic)
At the start: 7 parts, among them J3 SWD_UART, U2 STM32G0B1KxTxN

Commit message: fix schematic
Parts:
- renumbered C7 to C10, C3 to C6, C4 to C7, C5 to C8, C6 to C9, J3 to J12, U2 to U4
Changed lines of the file:
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@@
   (symbol (lib_id "Connector_Generic:Conn_02x05_Odd_Even") (at 200.66 128.27 0) (unit 1)
     (in_bom yes) (on_board yes)
-    (property "Reference" "J3" (id 0) (at 201.93 117.6782 0))
+    (property "Reference" "J12" (id 0) (at 201.93 117.6782 0))
     (property "Value" "SWD_UART" (id 1) (at 201.93 119.9896 0))
     (property "Footprint" "Connector_PinHeader_1.27mm:PinHeader_2x05_P1.27mm_Vertical_SMD" (id 2) (at 200.66 128.27 0)
@@
   (symbol (lib_id "power:+3V3") (at 191.77 121.92 0) (unit 1)
     (in_bom yes) (on_board yes)
-    (property "Reference" "#PWR015" (id 0) (at 191.77 125.73 0)
+    (property "Reference" "#PWR027" (id 0) (at 191.77 125.73 0)
       (effects (font (size 1.27 1.27)) hide)
     )
@@
   (symbol (lib_id "power:GND") (at 191.77 134.62 0) (unit 1)
     (in_bom yes) (on_board yes)
-    (property "Reference" "#PWR016" (id 0) (at 191.77 140.97 0)
+    (property "Reference" "#PWR028" (id 0) (at 191.77 140.97 0)
       (effects (font (size 1.27 1.27)) hide)
     )
@@
   (symbol (lib_id "extraparts:STM32G0B1KxTxN") (at 147.32 104.14 0) (unit 1)
     (in_bom yes) (on_board yes)
-    (property "Reference" "U2" (id 0) (at 165.1 77.47 0))
+    (property "Reference" "U4" (id 0) (at 165.1 77.47 0))
     (property "Value" "STM32G0B1KxTxN" (id 1) (at 171.45 80.01 0))
     (property "Footprint" "Package_QFP:LQFP-32_7x7mm_P0.8mm" (id 2) (at 147.32 59.69 0)
@@
   (symbol (lib_id "Device:C_Small") (at 152.4 66.04 0) (unit 1)
     (in_bom yes) (on_board yes)
-    (property "Reference" "C4" (id 0) (at 154.7368 64.8716 0)
+    (property "Reference" "C7" (id 0) (at 154.7368 64.8716 0)
       (effects (font (size 1.27 1.27)) (justify left))
     )
@@
   (symbol (lib_id "Device:C_Small") (at 161.29 66.04 0) (unit 1)
     (in_bom yes) (on_board yes)
-    (property "Reference" "C5" (id 0) (at 163.6268 64.8716 0)
+    (property "Reference" "C8" (id 0) (at 163.6268 64.8716 0)
       (effects (font (size 1.27 1.27)) (justify left))
     )
@@
   (symbol (lib_id "Device:C_Small") (at 170.18 66.04 0) (unit 1)
     (in_bom yes) (on_board yes)
-    (property "Reference" "C6" (id 0) (at 172.5168 64.8716 0)
+    (property "Reference" "C9" (id 0) (at 172.5168 64.8716 0)
       (effects (font (size 1.27 1.27)) (justify left))
     )
@@
   (symbol (lib_id "Device:C_Small") (at 179.07 66.04 0) (unit 1)
     (in_bom yes) (on_board yes)
-    (property "Reference" "C7" (id 0) (at 181.4068 64.8716 0)
+    (property "Reference" "C10" (id 0) (at 181.4068 64.8716 0)
       (effects (font (size 1.27 1.27)) (justify left))
     )
@@
   (symbol (lib_id "power:+3V3") (at 179.07 62.23 0) (unit 1)
     (in_bom yes) (on_board yes)
-    (property "Reference" "#PWR013" (id 0) (at 179.07 66.04 0)
+    (property "Reference" "#PWR025" (id 0) (at 179.07 66.04 0)
       (effects (font (size 1.27 1.27)) hide)
     )
@@
   (symbol (lib_id "power:GND") (at 179.07 69.85 0) (unit 1)
     (in_bom yes) (on_board yes)
-    (property "Reference" "#PWR014" (id 0) (at 179.07 76.2 0)
+    (property "Reference" "#PWR026" (id 0) (at 179.07 76.2 0)
       (effects (font (size 1.27 1.27)) hide)
     )
@@
   (symbol (lib_id "power:GND") (at 147.32 134.62 0) (unit 1)
     (in_bom yes) (on_board yes)
-    (property "Reference" "#PWR012" (id 0) (at 147.32 140.97 0)
+    (property "Reference" "#PWR024" (id 0) (at 147.32 140.97 0)
       (effects (font (size 1.27 1.27)) hide)
     )
@@
   (symbol (lib_id "Device:C_Small") (at 115.57 82.55 0) (unit 1)
     (in_bom yes) (on_board yes)
-    (property "Reference" "C3" (id 0) (at 117.9068 81.3816 0)
+    (property "Reference" "C6" (id 0) (at 117.9068 81.3816 0)
       (effects (font (size 1.27 1.27)) (justify left))
     )
@@
   (symbol (lib_id "power:GND") (at 115.57 86.36 0) (unit 1)
     (in_bom yes) (on_board yes)
-    (property "Reference" "#PWR011" (id 0) (at 115.57 92.71 0)
-      (effects (font (size 1.27 1.27)) hide)
-    )
+    (property "Reference" "#PWR023" (id 0) (at 115.57 92.71 0)
+      (effects (font (size 1.27 1.27)) hide)
+    )
