File: RoboSub/SidePlaneA/SidePlaneA.kicad_sch (KiCad schematic)
At the start: 40 parts, among them J1 CAN, J10 Conn_01x03, J11 Conn_01x03, J12 Conn_01x03, J2 CAN, J4 Conn_01x03, J5 Conn_01x03, J6 Conn_01x03, J7 Conn_01x03, J8 Conn_01x03, J9 Conn_01x03, SW1 DBG2, SW2 DBG1, SW3 RST, U3 ENS210

Commit message: modifications to footprints
Parts:
- C10, C11, C12, C13, C14, C15, C16, C8, C9: footprint (none) -> Capacitor_SMD:C_1206_3216Metric
- R4, R5: footprint (none) -> Resistor_SMD:R_0603_1608Metric
Changed lines of the file:
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@@
       (effects (font (size 1.27 1.27)) (justify left))
     )
-    (property "Footprint" "" (id 2) (at 116.5352 31.75 0)
+    (property "Footprint" "Capacitor_SMD:C_1206_3216Metric" (id 2) (at 116.5352 31.75 0)
       (effects (font (size 1.27 1.27)) hide)
     )
@@
       (effects (font (size 1.27 1.27)) (justify left))
     )
-    (property "Footprint" "" (id 2) (at 62.992 85.09 90)
+    (property "Footprint" "Resistor_SMD:R_0603_1608Metric" (id 2) (at 62.992 85.09 90)
       (effects (font (size 1.27 1.27)) hide)
     )
@@
       (effects (font (size 1.27 1.27)) (justify left))
     )
-    (property "Footprint" "" (id 2) (at 147.0152 31.75 0)
+    (property "Footprint" "Capacitor_SMD:C_1206_3216Metric" (id 2) (at 147.0152 31.75 0)
       (effects (font (size 1.27 1.27)) hide)
     )
@@
       (effects (font (size 1.27 1.27)) (justify left))
     )
-    (property "Footprint" "" (id 2) (at 209.2452 31.75 0)
+    (property "Footprint" "Capacitor_SMD:C_1206_3216Metric" (id 2) (at 209.2452 31.75 0)
       (effects (font (size 1.27 1.27)) hide)
     )
@@
       (effects (font (size 1.27 1.27)) (justify left))
     )
-    (property "Footprint" "" (id 2) (at 84.7852 80.01 0)
+    (property "Footprint" "Capacitor_SMD:C_1206_3216Metric" (id 2) (at 84.7852 80.01 0)
       (effects (font (size 1.27 1.27)) hide)
     )
@@
       (effects (font (size 1.27 1.27)) (justify left))
     )
-    (property "Footprint" "" (id 2) (at 86.0552 31.75 0)
+    (property "Footprint" "Capacitor_SMD:C_1206_3216Metric" (id 2) (at 86.0552 31.75 0)
       (effects (font (size 1.27 1.27)) hide)
     )
@@
     (property "Reference" "R5" (id 0) (at 77.47 83.82 0))
     (property "Value" "2.2k" (id 1) (at 77.47 86.36 0))
-    (property "Footprint" "" (id 2) (at 71.882 85.09 90)
+    (property "Footprint" "Resistor_SMD:R_0603_1608Metric" (id 2) (at 71.882 85.09 90)
       (effects (font (size 1.27 1.27)) hide)
     )
@@
       (effects (font (size 1.27 1.27)) (justify left))
     )
-    (property "Footprint" "" (id 2) (at 23.8252 31.75 0)
+    (property "Footprint" "Capacitor_SMD:C_1206_3216Metric" (id 2) (at 23.8252 31.75 0)
       (effects (font (size 1.27 1.27)) hide)
     )
@@
       (effects (font (size 1.27 1.27)) (justify left))
     )
-    (property "Footprint" "" (id 2) (at 177.4952 31.75 0)
+    (property "Footprint" "Capacitor_SMD:C_1206_3216Metric" (id 2) (at 177.4952 31.75 0)
       (effects (font (size 1.27 1.27)) hide)
     )
@@
       (effects (font (size 1.27 1.27)) (justify left))
     )
-    (property "Footprint" "" (id 2) (at 239.7252 31.75 0)
+    (property "Footprint" "Capacitor_SMD:C_1206_3216Metric" (id 2) (at 239.7252 31.75 0)
       (effects (font (size 1.27 1.27)) hide)
     )
@@
       (effects (font (size 1.27 1.27)) (justify left))
     )
-    (property "Footprint" "" (id 2) (at 54.3052 31.75 0)
+    (property "Footprint" "Capacitor_SMD:C_1206_3216Metric" (id 2) (at 54.3052 31.75 0)
       (effects (font (size 1.27 1.27)) hide)
     )
@@
     )
     (path "/b379ba47-de8b-4ced-95e6-e0b4100e84ba"
-      (reference "C8") (unit 1) (value "100n") (footprint "")
+      (reference "C8") (unit 1) (value "100n") (footprint "Capacitor_SMD:C_1206_3216Metric")
     )
     (path "/f893a184-5f7e-49ff-8b9a-8767b7e15b6d"
-      (reference "C9") (unit 1) (value "100n") (footprint "")
+      (reference "C9") (unit 1) (value "100n") (footprint "Capacitor_SMD:C_1206_3216Metric")
     )
     (path "/9a7d1f63-215d-4229-bf65-5c73ebd69d55"
-      (reference "C10") (unit 1) (value "100n") (footprint "")
+      (reference "C10") (unit 1) (value "100n") (footprint "Capacitor_SMD:C_1206_3216Metric")
     )
     (path "/a506be7c-e4d2-46b7-971f-e80dde1b2c42"
-      (reference "C11") (unit 1) (value "100n") (footprint "")
+      (reference "C11") (unit 1) (value "100n") (footprint "Capacitor_SMD:C_1206_3216Metric")
     )
     (path "/260064d3-eb78-4f3a-b377-252f750f76b2"
-      (reference "C12") (unit 1) (value "100n") (footprint "")
+      (reference "C12") (unit 1) (value "100n") (footprint "Capacitor_SMD:C_1206_3216Metric")
     )
     (path "/486da808-0693-4432-8336-008cae73a896"
-      (reference "C13") (unit 1) (value "100n") (footprint "")
+      (reference "C13") (unit 1) (value "100n") (footprint "Capacitor_SMD:C_1206_3216Metric")
     )
     (path "/c9326539-fb62-40cb-b63d-ef82e7793ede"
-      (reference "C14") (unit 1) (value "100n") (footprint "")
+      (reference "C14") (unit 1) (value "100n") (footprint "Capacitor_SMD:C_1206_3216Metric")
     )
     (path "/5b41a86b-7b57-43f1-b57b-9960051434db"
-      (reference "C15") (unit 1) (value "100n") (footprint "")
+      (reference "C15") (unit 1) (value "100n") (footprint "Capacitor_SMD:C_1206_3216Metric")
     )
     (path "/dbcd87e6-956e-40b7-937c-0f9b8b346268"
-      (reference "C16") (unit 1) (value "100n") (footprint "")
+      (reference "C16") (unit 1) (value "100n") (footprint "Capacitor_SMD:C_1206_3216Metric")
     )
     (path "/00000000-0000-0000-0000-00005e635a64"
@@
     )
     (path "/383eef67-c4c1-45aa-923b-83b59d1c3921"
-      (reference "R4") (unit 1) (value "2.2k") (footprint "")
+      (reference "R4") (unit 1) (value "2.2k") (footprint "Resistor_SMD:R_0603_1608Metric")
     )
     (path "/af5910e5-99b2-462c-a107-bfacfddeaa0d"
-      (reference "R5") (unit 1) (value "2.2k") (footprint "")
+      (reference "R5") (unit 1) (value "2.2k") (footprint "Resistor_SMD:R_0603_1608Metric")
     )
     (path "/00000000-0000-0000-0000-00005e62fb71"

Commit message: fix schematic
Parts:
- removed C10, C11, C12, C13, C14, C15, C16, C8, C9: 100n, Capacitor_SMD:C_1206_3216Metric, symbol Device:C
- removed D2, D3, D4, D5, D6, D7, D8, D9: WS2812B, LED_SMD:LED_WS2812B_PLCC4_5.0x5.0mm_P3.2mm, symbol LED:WS2812B
- removed J12: Conn_01x03, symbol Connector_Generic:Conn_01x03
- removed R4, R5: 2.2k, Resistor_SMD:R_0603_1608Metric, symbol Device:R
- removed U3: ENS210, Package_DFN_QFN:AMS_QFN-4-1EP_2x2mm_P0.95mm_EP0.7x1.6mm, symbol Sensor_Humidity:ENS210
- added C1: 100n, symbol Device:C_Small
- added C2, C3: 10u, Capacitor_SMD:C_0805_2012Metric, symbol Device:C_Small
- added J9: WS2812B, symbol Connector_Generic:Conn_01x03
- added R1, R2: 2k2, symbol Device:R_Small
- added U1: SHT30-DIS, Sensor_Humidity:Sensirion_DFN-8-1EP_2.5x2.5mm_P0.5mm_EP1.1x1.7mm, symbol Sensor_Humidity:SHT30-DIS
- added U2: R-78E5.0-1.0, Converter_DCDC:Converter_DCDC_RECOM_R-78E-0.5_THT, symbol Regulator_Switching:R-78E5.0-1.0
- J1, J2: value CAN -> Spine
- J10: value Conn_01x03 -> motor4_out
- J11: value Conn_01x03 -> motor4_in
- J3: renamed from J4; value Conn_01x03 -> motor1_out
- J4: renamed from J5; value Conn_01x03 -> motor1_in
- J5: renamed from J6; value Conn_01x03 -> motor2_out
- J6: renamed from J7; value Conn_01x03 -> motor2_in
- J7: renamed from J8; value Conn_01x03 -> motor3_out
- J8: renamed from J9; value Conn_01x03 -> motor3_in
- renumbered R1 to R3, R2 to R4, R3 to R5
Connections:
- net +12V: now also C2.2, U2.1 (IN)
- net +3V3: now also C1.2, R1.1, R2.1, U1.5 (VDD)
- net +5V: now also C3.1, J9.2 (Pin_2), U2.3 (OUT)
- net GND: now also C1.1, C2.1, C3.2, J9.1 (Pin_1), U1.2 (ADDR), U1.7 (R), U1.8 (VSS), U1.9 (VSS), U2.2 (GND)
- net SCL: now also R2.2, U1.4 (SCL)
- net SDA: now also R1.2, U1.1 (SDA)
- new net ws2812b_dout: J9.3 (Pin_3)
- no-connect marks 0 -> 20
Other:
- added sheet WS2812B_1 (ws2812b.kicad_sch)
- added sheet WS2812B_2 (ws2812b.kicad_sch)
- added sheet WS2812B_3 (ws2812b.kicad_sch)
- added sheet WS2812B_4 (ws2812b.kicad_sch)
- added sheet WS2812B_5 (ws2812b.kicad_sch)
- added sheet WS2812B_6 (ws2812b.kicad_sch)
- added sheet WS2812B_7 (ws2812b.kicad_sch)
- added sheet WS2812B_8 (ws2812b.kicad_sch)
- note added: "I2C2"
- note added: "Motor Passthrough"
- note added: "SPI1_MOSI"
- note removed: "2 connectors for daisy-chaining"
- note removed: "CAN connector provides 12v and 3v3 too"
- note removed: "contains the micro and debug connector keep caps close to micro"
- note removed: "switches and LED for debugging feel free to move/remove"
- moved on the sheet: D1, F1, F2, J1, J10, J11, J2, J3, J4, J5, J6, J7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
