File: RoboSub/Backplane/Backplane.kicad_sch (KiCad schematic)
At the start: 28 parts, among them J1 BatteryIn, J10 motor4, J11 motor5, J12 motor6, J13 JetsonPWR, J14 JetsonCAN, J2 I2C, J3 Spine, J4 Spine, J5 Spine, J6 IMU, J7 motor1, J8 motor2, J9 motor3, M1 ESCB, M2 ESCB, M3 ESCB, M4 ESCB, M5 ESCB, M6 ESCB, SW1 DBG2, SW2 DBG1, SW3 RST

Commit message: add libs
Parts:
- added R4, R5: 2k2, Resistor_SMD:R_0603_1608Metric, symbol Device:R_Small
- J1: footprint extraparts:Molex_SuperSabre_Vert_2pin -> (none)
- J14: footprint (none) -> extraparts:Molex_DuraClik_Vert_3pin
Connections:
- net +3V3: now also R4.1, R5.1
- net SCL: now also R4.2
- net SDA: now also R5.2
Changed lines of the file:
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@@
+    (stroke (width 0) (type default) (color 0 0 0 0))
+  )
+  (wire (pts (xy 80.01 85.09) (xy 95.885 85.09))
     (stroke (width 0) (type default) (color 0 0 0 0))
   )
@@
     (stroke (width 0) (type default) (color 0 0 0 0))
   )
+  (wire (pts (xy 80.01 87.63) (xy 102.235 87.63))
+    (stroke (width 0) (type default) (color 0 0 0 0))
+  )
   (wire (pts (xy 213.995 52.07) (xy 213.995 53.34))
     (stroke (width 0) (type default) (color 0 0 0 0))
@@
     (stroke (width 0) (type default) (color 0 0 0 0))
   )
+  (wire (pts (xy 95.885 78.74) (xy 95.885 79.375))
+    (stroke (width 0) (type default) (color 0 0 0 0))
+  )
   (wire (pts (xy 49.53 132.715) (xy 49.53 117.475))
     (stroke (width 0) (type default) (color 0 0 0 0))
@@
     (stroke (width 0) (type default) (color 0 0 0 0))
   )
+  (wire (pts (xy 102.235 78.74) (xy 102.235 79.375))
+    (stroke (width 0) (type default) (color 0 0 0 0))
+  )
   (wire (pts (xy 253.365 132.715) (xy 252.095 132.715))
     (stroke (width 0) (type default) (color 0 0 0 0))
@@
     (stroke (width 0) (type default) (color 0 0 0 0))
   )
+  (wire (pts (xy 102.235 87.63) (xy 102.235 84.455))
+    (stroke (width 0) (type default) (color 0 0 0 0))
+  )
   (wire (pts (xy 43.18 125.095) (xy 45.72 125.095))
     (stroke (width 0) (type default) (color 0 0 0 0))
@@
   )
   (wire (pts (xy 170.815 52.07) (xy 170.815 53.34))
+    (stroke (width 0) (type default) (color 0 0 0 0))
+  )
+  (wire (pts (xy 95.885 85.09) (xy 95.885 84.455))
     (stroke (width 0) (type default) (color 0 0 0 0))
   )
@@
     (property "Reference" "J14" (id 0) (at 258.445 141.605 0))
     (property "Value" "JetsonCAN" (id 1) (at 265.43 146.685 0))
-    (property "Footprint" "" (id 2) (at 258.445 146.685 0)
+    (property "Footprint" "extraparts:Molex_DuraClik_Vert_3pin" (id 2) (at 258.445 146.685 0)
       (effects (font (size 1.27 1.27)) hide)
     )
@@
     (pin "6")
   )
+  (symbol (lib_id "power:+3V3") (at 102.235 78.74 0) (unit 1)
+    (in_bom yes) (on_board yes)
+    (property "Reference" "#PWR0102" (id 0) (at 102.235 82.55 0)
+      (effects (font (size 1.27 1.27)) hide)
+    )
+    (property "Value" "+3V3" (id 1) (at 102.235 74.93 0))
+    (property "Footprint" "" (id 2) (at 102.235 78.74 0)
+      (effects (font (size 1.27 1.27)) hide)
+    )
+    (property "Datasheet" "" (id 3) (at 102.235 78.74 0)
+      (effects (font (size 1.27 1.27)) hide)
+    )
+    (pin "1")
+  )
   (symbol (lib_id "power:GND") (at 44.45 68.58 0) (mirror y) (unit 1)
     (in_bom yes) (on_board yes)
@@
     (pin "1")
   )
+  (symbol (lib_id "Device:R_Small") (at 95.885 81.915 0) (unit 1)
+    (in_bom yes) (on_board yes) (fields_autoplaced)
+    (property "Reference" "R4" (id 0) (at 97.3836 81.0065 0)
+      (effects (font (size 1.27 1.27)) (justify left))
+    )
+    (property "Value" "2k2" (id 1) (at 97.3836 83.7816 0)
+      (effects (font (size 1.27 1.27)) (justify left))
+    )
+    (property "Footprint" "Resistor_SMD:R_0603_1608Metric" (id 2) (at 95.885 81.915 0)
+      (effects (font (size 1.27 1.27)) hide)
+    )
+    (property "Datasheet" "~" (id 3) (at 95.885 81.915 0)
+      (effects (font (size 1.27 1.27)) hide)
+    )
+    (pin "1")
+    (pin "2")
+  )
   (symbol (lib_id "Connector_Generic:Conn_01x03") (at 216.535 46.99 90) (unit 1)
     (in_bom yes) (on_board yes)
@@
     (pin "4")
   )
+  (symbol (lib_id "power:+3V3") (at 95.885 78.74 0) (unit 1)
+    (in_bom yes) (on_board yes)
+    (property "Reference" "#PWR0101" (id 0) (at 95.885 82.55 0)
+      (effects (font (size 1.27 1.27)) hide)
+    )
+    (property "Value" "+3V3" (id 1) (at 95.885 74.93 0))
+    (property "Footprint" "" (id 2) (at 95.885 78.74 0)
+      (effects (font (size 1.27 1.27)) hide)
+    )
+    (property "Datasheet" "" (id 3) (at 95.885 78.74 0)
+      (effects (font (size 1.27 1.27)) hide)
+    )
+    (pin "1")
+  )
   (symbol (lib_id "power:GND") (at 144.145 69.85 270) (unit 1)
     (in_bom yes) (on_board yes)
@@
     (property "Reference" "J1" (id 0) (at 38.1 62.23 0))
     (property "Value" "BatteryIn" (id 1) (at 32.385 66.04 0))
-    (property "Footprint" "extraparts:Molex_SuperSabre_Vert_2pin" (id 2) (at 38.1 67.31 0)
+    (property "Footprint" "" (id 2) (at 38.1 67.31 0)
       (effects (font (size 1.27 1.27)) hide)
     )
@@
     )
     (pin "1")
+  )
+  (symbol (lib_id "Device:R_Small") (at 102.235 81.915 0) (unit 1)
+    (in_bom yes) (on_board yes) (fields_autoplaced)
+    (property "Reference" "R5" (id 0) (at 103.7336 81.0065 0)
+      (effects (font (size 1.27 1.27)) (justify left))
+    )
+    (property "Value" "2k2" (id 1) (at 103.7336 83.7816 0)
+      (effects (font (size 1.27 1.27)) (justify left))
+    )
+    (property "Footprint" "Resistor_SMD:R_0603_1608Metric" (id 2) (at 102.235 81.915 0)
+      (effects (font (size 1.27 1.27)) hide)
+    )
+    (property "Datasheet" "~" (id 3) (at 102.235 81.915 0)
+      (effects (font (size 1.27 1.27)) hide)
+    )
+    (pin "1")
+    (pin "2")
   )
   (symbol (lib_id "Connector_Generic:Conn_01x04") (at 38.1 85.09 180) (unit 1)
@@
       (reference "#PWR041") (unit 1) (value "GND") (footprint "")
     )
+    (path "/aa97fd18-7573-4c36-b186-394e7d270518"
+      (reference "#PWR0101") (unit 1) (value "+3V3") (footprint "")
+    )
+    (path "/5302655e-adcd-494d-9861-53f4df5616e5"
+      (reference "#PWR0102") (unit 1) (value "+3V3") (footprint "")
+    )
     (path "/1be8059f-78fe-473a-9436-3e2c303393ac/d2898eb2-73b6-44c9-948c-0a712fbf2152"
       (reference "C1") (unit 1) (value "100n") (footprint "Capacitor_SMD:C_0603_1608Metric")
@@
     )
     (path "/c65e486c-e5df-495f-8f19-613bdaa7aadd"
-      (reference "J1") (unit 1) (value "BatteryIn") (footprint "extraparts:Molex_SuperSabre_Vert_2pin")
+      (reference "J1") (unit 1) (value "BatteryIn") (footprint "")
     )
     (path "/e5401138-527e-4a0b-b275-9e5fd17d10ae"
@@
     )
     (path "/491b7a53-831c-4e3a-ae32-6aec78235d42"
-      (reference "J14") (unit 1) (value "JetsonCAN") (footprint "")
+      (reference "J14") (unit 1) (value "JetsonCAN") (footprint "extraparts:Molex_DuraClik_Vert_3pin")
     )
     (path "/02a592e2-7d43-4770-a734-d28fb2a73cb2/c313b079-be60-457c-9f7e-a25ce21cd0f4"
@@
       (reference "R3") (unit 1) (value "47") (footprint "Resistor_SMD:R_0603_1608Metric")
     )
+    (path "/9cf37ab0-58d2-419a-9c76-4836af0b31df"
+      (reference "R4") (unit 1) (value "2k2") (footprint "Resistor_SMD:R_0603_1608Metric")
+    )
+    (path "/daf9da28-0f62-4030-a96d-6aecd6fce210"
+      (reference "R5") (unit 1) (value "2k2") (footprint "Resistor_SMD:R_0603_1608Metric")
+    )
     (path "/322cbbc5-0482-4f79-8ee0-e1fed12c0b59"

Commit message: layout placement done, haven't connect nets
Parts:
- J1: footprint (none) -> extraparts:Molex_SuperSabre_Vert_2pin
- J10, J11, J12, J7, J8, J9: footprint (none) -> extraparts:Molex_UltraFit_RH_3pin
- M1, M2, M3, M4, M5, M6: footprint (none) -> urbparts:ESCB_mate
Changed lines of the file:
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@@
       (effects (font (size 1.27 1.27)) (justify left))
     )
-    (property "Footprint" "" (id 2) (at 170.815 60.96 0)
+    (property "Footprint" "urbparts:ESCB_mate" (id 2) (at 170.815 60.96 0)
       (effects (font (size 1.27 1.27)) hide)
     )
@@
       (effects (font (size 1.27 1.27)) (justify right))
     )
-    (property "Footprint" "" (id 2) (at 147.955 46.99 0)
+    (property "Footprint" "extraparts:Molex_UltraFit_RH_3pin" (id 2) (at 147.955 46.99 0)
       (effects (font (size 1.27 1.27)) hide)
     )
@@
       (effects (font (size 1.27 1.27)) (justify left))
     )
-    (property "Footprint" "" (id 2) (at 216.535 60.96 0)
+    (property "Footprint" "urbparts:ESCB_mate" (id 2) (at 216.535 60.96 0)
       (effects (font (size 1.27 1.27)) hide)
     )
@@
       (effects (font (size 1.27 1.27)) (justify right))
     )
-    (property "Footprint" "" (id 2) (at 193.675 46.99 0)
+    (property "Footprint" "extraparts:Molex_UltraFit_RH_3pin" (id 2) (at 193.675 46.99 0)
       (effects (font (size 1.27 1.27)) hide)
     )
@@
       (effects (font (size 1.27 1.27)) (justify right))
     )
-    (property "Footprint" "" (id 2) (at 125.095 46.99 0)
+    (property "Footprint" "extraparts:Molex_UltraFit_RH_3pin" (id 2) (at 125.095 46.99 0)
       (effects (font (size 1.27 1.27)) hide)
     )
@@
       (effects (font (size 1.27 1.27)) (justify left))
     )
-    (property "Footprint" "" (id 2) (at 193.675 60.96 0)
+    (property "Footprint" "urbparts:ESCB_mate" (id 2) (at 193.675 60.96 0)
       (effects (font (size 1.27 1.27)) hide)
     )
@@
       (effects (font (size 1.27 1.27)) (justify left))
     )
-    (property "Footprint" "" (id 2) (at 147.955 60.96 0)
+    (property "Footprint" "urbparts:ESCB_mate" (id 2) (at 147.955 60.96 0)
       (effects (font (size 1.27 1.27)) hide)
     )
@@
       (effects (font (size 1.27 1.27)) (justify right))
     )
-    (property "Footprint" "" (id 2) (at 170.815 46.99 0)
+    (property "Footprint" "extraparts:Molex_UltraFit_RH_3pin" (id 2) (at 170.815 46.99 0)
       (effects (font (size 1.27 1.27)) hide)
     )
@@
       (effects (font (size 1.27 1.27)) (justify right))
     )
-    (property "Footprint" "" (id 2) (at 216.535 46.99 0)
+    (property "Footprint" "extraparts:Molex_UltraFit_RH_3pin" (id 2) (at 216.535 46.99 0)
       (effects (font (size 1.27 1.27)) hide)
     )
@@
       (effects (font (size 1.27 1.27)) (justify right))
     )
-    (property "Footprint" "" (id 2) (at 239.395 46.99 0)
+    (property "Footprint" "extraparts:Molex_UltraFit_RH_3pin" (id 2) (at 239.395 46.99 0)
       (effects (font (size 1.27 1.27)) hide)
     )
@@
     (property "Reference" "J1" (id 0) (at 38.1 62.23 0))
     (property "Value" "BatteryIn" (id 1) (at 32.385 66.04 0))
-    (property "Footprint" "" (id 2) (at 38.1 67.31 0)
+    (property "Footprint" "extraparts:Molex_SuperSabre_Vert_2pin" (id 2) (at 38.1 67.31 0)
       (effects (font (size 1.27 1.27)) hide)
     )
@@
       (effects (font (size 1.27 1.27)) (justify left))
     )
-    (property "Footprint" "" (id 2) (at 125.095 60.96 0)
+    (property "Footprint" "urbparts:ESCB_mate" (id 2) (at 125.095 60.96 0)
       (effects (font (size 1.27 1.27)) hide)
     )
@@
       (effects (font (size 1.27 1.27)) (justify left))
     )
-    (property "Footprint" "" (id 2) (at 239.395 60.96 0)
+    (property "Footprint" "urbparts:ESCB_mate" (id 2) (at 239.395 60.96 0)
       (effects (font (size 1.27 1.27)) hide)
     )
@@
     )
     (path "/c65e486c-e5df-495f-8f19-613bdaa7aadd"
-      (reference "J1") (unit 1) (value "BatteryIn") (footprint "")
+      (reference "J1") (unit 1) (value "BatteryIn") (footprint "extraparts:Molex_SuperSabre_Vert_2pin")
     )
     (path "/e5401138-527e-4a0b-b275-9e5fd17d10ae"
@@
     )
     (path "/610e608d-da82-4b55-bcff-67e240ba053d"
-      (reference "J7") (unit 1) (value "motor1") (footprint "")
+      (reference "J7") (unit 1) (value "motor1") (footprint "extraparts:Molex_UltraFit_RH_3pin")
     )
     (path "/455f91ae-43a8-4341-86c1-7bc2916e1adb"
-      (reference "J8") (unit 1) (value "motor2") (footprint "")
+      (reference "J8") (unit 1) (value "motor2") (footprint "extraparts:Molex_UltraFit_RH_3pin")
     )
     (path "/9afc22d5-a90e-44a8-a232-f12a91ea8339"
-      (reference "J9") (unit 1) (value "motor3") (footprint "")
+      (reference "J9") (unit 1) (value "motor3") (footprint "extraparts:Molex_UltraFit_RH_3pin")
     )
     (path "/6082bf26-08e6-4ef7-92f1-102a208ed637"
-      (reference "J10") (unit 1) (value "motor4") (footprint "")
+      (reference "J10") (unit 1) (value "motor4") (footprint "extraparts:Molex_UltraFit_RH_3pin")
     )
     (path "/9e3de139-600a-4bc8-816f-dbae59619d00"
-      (reference "J11") (unit 1) (value "motor5") (footprint "")
+      (reference "J11") (unit 1) (value "motor5") (footprint "extraparts:Molex_UltraFit_RH_3pin")
     )
     (path "/b29081f8-d144-4360-bd1b-03db2a7e1fa0"
-      (reference "J12") (unit 1) (value "motor6") (footprint "")
+      (reference "J12") (unit 1) (value "motor6") (footprint "extraparts:Molex_UltraFit_RH_3pin")
     )
     (path "/9b006909-1d1a-4b82-a16a-11ac81f7af59"
@@
     )
     (path "/c6af5a2d-0f49-4897-86b4-9410a82b05dd"
-      (reference "M1") (unit 1) (value "ESCB") (footprint "")
+      (reference "M1") (unit 1) (value "ESCB") (footprint "urbparts:ESCB_mate")
     )
     (path "/885de0be-5aeb-48d6-81a8-ab24ce558efd"
-      (reference "M2") (unit 1) (value "ESCB") (footprint "")
+      (reference "M2") (unit 1) (value "ESCB") (footprint "urbparts:ESCB_mate")
     )
     (path "/4494a3fd-896d-41cf-89dc-0cb647ab771b"
-      (reference "M3") (unit 1) (value "ESCB") (footprint "")
+      (reference "M3") (unit 1) (value "ESCB") (footprint "urbparts:ESCB_mate")
     )
     (path "/71164ffa-28d5-491a-a718-ff41582d56c9"
-      (reference "M4") (unit 1) (value "ESCB") (footprint "")
+      (reference "M4") (unit 1) (value "ESCB") (footprint "urbparts:ESCB_mate")
     )
     (path "/51c27063-a7b5-43d9-8b12-cce911f99048"
-      (reference "M5") (unit 1) (value "ESCB") (footprint "")
+      (reference "M5") (unit 1) (value "ESCB") (footprint "urbparts:ESCB_mate")
     )
     (path "/eb783504-e86d-40b0-a442-16621c4c1f93"
-      (reference "M6") (unit 1) (value "ESCB") (footprint "")
+      (reference "M6") (unit 1) (value "ESCB") (footprint "urbparts:ESCB_mate")
     )
     (path "/ec28b849-8c86-4a4f-9bda-d2af97194ad6"

Commit message: first backplane layout commit
Parts:
- J1: footprint extraparts:Molex_SuperSabre_Vert_2pin -> urbparts:Conn_XT90
- J10, J11, J12, J7, J8, J9: footprint extraparts:Molex_UltraFit_RH_3pin -> extraparts:Molex_UltraFit_Vert_3pin
Changed lines of the file:
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@@
       (effects (font (size 1.27 1.27)) (justify right))
     )
-    (property "Footprint" "extraparts:Molex_UltraFit_RH_3pin" (id 2) (at 147.955 46.99 0)
+    (property "Footprint" "extraparts:Molex_UltraFit_Vert_3pin" (id 2) (at 147.955 46.99 0)
       (effects (font (size 1.27 1.27)) hide)
     )
@@
       (effects (font (size 1.27 1.27)) (justify right))
     )
-    (property "Footprint" "extraparts:Molex_UltraFit_RH_3pin" (id 2) (at 193.675 46.99 0)
+    (property "Footprint" "extraparts:Molex_UltraFit_Vert_3pin" (id 2) (at 193.675 46.99 0)
       (effects (font (size 1.27 1.27)) hide)
     )
@@
       (effects (font (size 1.27 1.27)) (justify right))
     )
-    (property "Footprint" "extraparts:Molex_UltraFit_RH_3pin" (id 2) (at 125.095 46.99 0)
+    (property "Footprint" "extraparts:Molex_UltraFit_Vert_3pin" (id 2) (at 125.095 46.99 0)
       (effects (font (size 1.27 1.27)) hide)
     )
@@
       (effects (font (size 1.27 1.27)) (justify right))
     )
-    (property "Footprint" "extraparts:Molex_UltraFit_RH_3pin" (id 2) (at 170.815 46.99 0)
+    (property "Footprint" "extraparts:Molex_UltraFit_Vert_3pin" (id 2) (at 170.815 46.99 0)
       (effects (font (size 1.27 1.27)) hide)
     )
@@
       (effects (font (size 1.27 1.27)) (justify right))
     )
-    (property "Footprint" "extraparts:Molex_UltraFit_RH_3pin" (id 2) (at 216.535 46.99 0)
+    (property "Footprint" "extraparts:Molex_UltraFit_Vert_3pin" (id 2) (at 216.535 46.99 0)
       (effects (font (size 1.27 1.27)) hide)
     )
@@
       (effects (font (size 1.27 1.27)) (justify right))
     )
-    (property "Footprint" "extraparts:Molex_UltraFit_RH_3pin" (id 2) (at 239.395 46.99 0)
+    (property "Footprint" "extraparts:Molex_UltraFit_Vert_3pin" (id 2) (at 239.395 46.99 0)
       (effects (font (size 1.27 1.27)) hide)
     )
@@
     (property "Reference" "J1" (id 0) (at 38.1 62.23 0))
     (property "Value" "BatteryIn" (id 1) (at 32.385 66.04 0))
-    (property "Footprint" "extraparts:Molex_SuperSabre_Vert_2pin" (id 2) (at 38.1 67.31 0)
+    (property "Footprint" "urbparts:Conn_XT90" (id 2) (at 38.1 67.31 0)
       (effects (font (size 1.27 1.27)) hide)
     )
@@
     )
     (path "/c65e486c-e5df-495f-8f19-613bdaa7aadd"
-      (reference "J1") (unit 1) (value "BatteryIn") (footprint "extraparts:Molex_SuperSabre_Vert_2pin")
+      (reference "J1") (unit 1) (value "BatteryIn") (footprint "urbparts:Conn_XT90")
     )
     (path "/e5401138-527e-4a0b-b275-9e5fd17d10ae"
@@
     )
     (path "/610e608d-da82-4b55-bcff-67e240ba053d"
-      (reference "J7") (unit 1) (value "motor1") (footprint "extraparts:Molex_UltraFit_RH_3pin")
+      (reference "J7") (unit 1) (value "motor1") (footprint "extraparts:Molex_UltraFit_Vert_3pin")
     )
     (path "/455f91ae-43a8-4341-86c1-7bc2916e1adb"
-      (reference "J8") (unit 1) (value "motor2") (footprint "extraparts:Molex_UltraFit_RH_3pin")
+      (reference "J8") (unit 1) (value "motor2") (footprint "extraparts:Molex_UltraFit_Vert_3pin")
     )
     (path "/9afc22d5-a90e-44a8-a232-f12a91ea8339"
-      (reference "J9") (unit 1) (value "motor3") (footprint "extraparts:Molex_UltraFit_RH_3pin")
+      (reference "J9") (unit 1) (value "motor3") (footprint "extraparts:Molex_UltraFit_Vert_3pin")
     )
     (path "/6082bf26-08e6-4ef7-92f1-102a208ed637"
-      (reference "J10") (unit 1) (value "motor4") (footprint "extraparts:Molex_UltraFit_RH_3pin")
+      (reference "J10") (unit 1) (value "motor4") (footprint "extraparts:Molex_UltraFit_Vert_3pin")
     )
     (path "/9e3de139-600a-4bc8-816f-dbae59619d00"
-      (reference "J11") (unit 1) (value "motor5") (footprint "extraparts:Molex_UltraFit_RH_3pin")
+      (reference "J11") (unit 1) (value "motor5") (footprint "extraparts:Molex_UltraFit_Vert_3pin")
     )
     (path "/b29081f8-d144-4360-bd1b-03db2a7e1fa0"
-      (reference "J12") (unit 1) (value "motor6") (footprint "extraparts:Molex_UltraFit_RH_3pin")
+      (reference "J12") (unit 1) (value "motor6") (footprint "extraparts:Molex_UltraFit_Vert_3pin")
     )
     (path "/9b006909-1d1a-4b82-a16a-11ac81f7af59"

Commit message: made changes to blackplane layout second commit
Parts:
- J10, J11, J12, J7, J8, J9: footprint extraparts:Molex_UltraFit_Vert_3pin -> extraparts:Molex_UltraFit_KP_Vert_3pin
Changed lines of the file:
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@@
       (effects (font (size 1.27 1.27)) (justify right))
     )
-    (property "Footprint" "extraparts:Molex_UltraFit_Vert_3pin" (id 2) (at 147.955 46.99 0)
+    (property "Footprint" "extraparts:Molex_UltraFit_KP_Vert_3pin" (id 2) (at 147.955 46.99 0)
       (effects (font (size 1.27 1.27)) hide)
     )
@@
       (effects (font (size 1.27 1.27)) (justify right))
     )
-    (property "Footprint" "extraparts:Molex_UltraFit_Vert_3pin" (id 2) (at 193.675 46.99 0)
+    (property "Footprint" "extraparts:Molex_UltraFit_KP_Vert_3pin" (id 2) (at 193.675 46.99 0)
       (effects (font (size 1.27 1.27)) hide)
     )
@@
       (effects (font (size 1.27 1.27)) (justify right))
     )
-    (property "Footprint" "extraparts:Molex_UltraFit_Vert_3pin" (id 2) (at 125.095 46.99 0)
+    (property "Footprint" "extraparts:Molex_UltraFit_KP_Vert_3pin" (id 2) (at 125.095 46.99 0)
       (effects (font (size 1.27 1.27)) hide)
     )
@@
       (effects (font (size 1.27 1.27)) (justify right))
     )
-    (property "Footprint" "extraparts:Molex_UltraFit_Vert_3pin" (id 2) (at 170.815 46.99 0)
+    (property "Footprint" "extraparts:Molex_UltraFit_KP_Vert_3pin" (id 2) (at 170.815 46.99 0)
       (effects (font (size 1.27 1.27)) hide)
     )
@@
       (effects (font (size 1.27 1.27)) (justify right))
     )
-    (property "Footprint" "extraparts:Molex_UltraFit_Vert_3pin" (id 2) (at 216.535 46.99 0)
+    (property "Footprint" "extraparts:Molex_UltraFit_KP_Vert_3pin" (id 2) (at 216.535 46.99 0)
       (effects (font (size 1.27 1.27)) hide)
     )
@@
       (effects (font (size 1.27 1.27)) (justify right))
     )
-    (property "Footprint" "extraparts:Molex_UltraFit_Vert_3pin" (id 2) (at 239.395 46.99 0)
+    (property "Footprint" "extraparts:Molex_UltraFit_KP_Vert_3pin" (id 2) (at 239.395 46.99 0)
       (effects (font (size 1.27 1.27)) hide)
     )
@@
     )
     (path "/610e608d-da82-4b55-bcff-67e240ba053d"
-      (reference "J7") (unit 1) (value "motor1") (footprint "extraparts:Molex_UltraFit_Vert_3pin")
+      (reference "J7") (unit 1) (value "motor1") (footprint "extraparts:Molex_UltraFit_KP_Vert_3pin")
     )
     (path "/455f91ae-43a8-4341-86c1-7bc2916e1adb"
-      (reference "J8") (unit 1) (value "motor2") (footprint "extraparts:Molex_UltraFit_Vert_3pin")
+      (reference "J8") (unit 1) (value "motor2") (footprint "extraparts:Molex_UltraFit_KP_Vert_3pin")
     )
     (path "/9afc22d5-a90e-44a8-a232-f12a91ea8339"
-      (reference "J9") (unit 1) (value "motor3") (footprint "extraparts:Molex_UltraFit_Vert_3pin")
+      (reference "J9") (unit 1) (value "motor3") (footprint "extraparts:Molex_UltraFit_KP_Vert_3pin")
     )
     (path "/6082bf26-08e6-4ef7-92f1-102a208ed637"
-      (reference "J10") (unit 1) (value "motor4") (footprint "extraparts:Molex_UltraFit_Vert_3pin")
+      (reference "J10") (unit 1) (value "motor4") (footprint "extraparts:Molex_UltraFit_KP_Vert_3pin")
     )
     (path "/9e3de139-600a-4bc8-816f-dbae59619d00"
-      (reference "J11") (unit 1) (value "motor5") (footprint "extraparts:Molex_UltraFit_Vert_3pin")
+      (reference "J11") (unit 1) (value "motor5") (footprint "extraparts:Molex_UltraFit_KP_Vert_3pin")
     )
     (path "/b29081f8-d144-4360-bd1b-03db2a7e1fa0"
-      (reference "J12") (unit 1) (value "motor6") (footprint "extraparts:Molex_UltraFit_Vert_3pin")
+      (reference "J12") (unit 1) (value "motor6") (footprint "extraparts:Molex_UltraFit_KP_Vert_3pin")
     )
     (path "/9b006909-1d1a-4b82-a16a-11ac81f7af59"
