File: RoboSub/Backplane/NOGGIN_Block.kicad_sch (KiCad schematic)
At the start: 7 parts

Commit message: fix schematic
Parts:
- gave numbers to parts that had none: 2
Changed lines of the file:
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@@
   (symbol (lib_id "power:GND") (at 90.17 82.55 0) (unit 1)
     (in_bom yes) (on_board yes)
-    (property "Reference" "#PWR?" (id 0) (at 90.17 88.9 0)
+    (property "Reference" "#PWR033" (id 0) (at 90.17 88.9 0)
       (effects (font (size 1.27 1.27)) hide)
     )
@@
   (symbol (lib_id "power:GND") (at 153.67 66.04 0) (unit 1)
     (in_bom yes) (on_board yes)
-    (property "Reference" "#PWR?" (id 0) (at 153.67 72.39 0)
+    (property "Reference" "#PWR036" (id 0) (at 153.67 72.39 0)
       (effects (font (size 1.27 1.27)) hide)
     )
@@
   (symbol (lib_id "power:+3V3") (at 166.37 118.11 0) (unit 1)
     (in_bom yes) (on_board yes)
-    (property "Reference" "#PWR?" (id 0) (at 166.37 121.92 0)
+    (property "Reference" "#PWR037" (id 0) (at 166.37 121.92 0)
       (effects (font (size 1.27 1.27)) hide)
     )
@@
   (symbol (lib_id "power:GND") (at 166.37 130.81 0) (unit 1)
     (in_bom yes) (on_board yes)
-    (property "Reference" "#PWR?" (id 0) (at 166.37 137.16 0)
+    (property "Reference" "#PWR038" (id 0) (at 166.37 137.16 0)
       (effects (font (size 1.27 1.27)) hide)
     )
@@
   (symbol (lib_id "extraparts:STM32G0B1KxTxN") (at 121.92 100.33 0) (unit 1)
     (in_bom yes) (on_board yes)
-    (property "Reference" "U?" (id 0) (at 139.7 73.66 0))
+    (property "Reference" "U2" (id 0) (at 139.7 73.66 0))
     (property "Value" "STM32G0B1KxTxN" (id 1) (at 146.05 76.2 0))
     (property "Footprint" "Package_QFP:LQFP-32_7x7mm_P0.8mm" (id 2) (at 121.92 55.88 0)
@@
   (symbol (lib_id "Connector_Generic:Conn_02x05_Odd_Even") (at 175.26 124.46 0) (unit 1)
     (in_bom yes) (on_board yes)
-    (property "Reference" "J?" (id 0) (at 176.53 113.8682 0))
+    (property "Reference" "J15" (id 0) (at 176.53 113.8682 0))
     (property "Value" "SWD_UART" (id 1) (at 176.53 116.1796 0))
     (property "Footprint" "Connector_PinHeader_1.27mm:PinHeader_2x05_P1.27mm_Vertical_SMD" (id 2) (at 175.26 124.46 0)
@@
   (symbol (lib_id "power:GND") (at 121.92 130.81 0) (unit 1)
     (in_bom yes) (on_board yes)
-    (property "Reference" "#PWR?" (id 0) (at 121.92 137.16 0)
+    (property "Reference" "#PWR034" (id 0) (at 121.92 137.16 0)
       (effects (font (size 1.27 1.27)) hide)
     )
@@
   (symbol (lib_id "power:+3V3") (at 153.67 58.42 0) (unit 1)
     (in_bom yes) (on_board yes)
-    (property "Reference" "#PWR?" (id 0) (at 153.67 62.23 0)
-      (effects (font (size 1.27 1.27)) hide)
-    )
+    (property "Reference" "#PWR035" (id 0) (at 153.67 62.23 0)
+      (effects (font (size 1.27 1.27)) hide)
+    )
