File: RoboSub/BMS/BMS.kicad_pcb (KiCad board)
At the start: 2 copper layers, 127.5 x 55.1 mm, 44 parts, among them J1 battery, J2 temp, J3 ExtPwrSw, J4 output, J5 CAN, J6 SWD_UART, K1 A3M1CSQ12VDC2, Q1 PMV28ENEA, SW1 DBG2, SW2 DBG1, SW3 RST, U1 R-785.0-1.0, U2 CZ3A07, U3 STM32G0B1KxTxN, U4 TCAN330G, U5 PCC, U6 AZ1117-3.3

Commit message: forgot to save some changes. Now up to date.
Routing:
- net /DBG2: track 11.9 -> 16.0 mm
- net /DBG1: track 9.48 -> 13.6 mm
- net GND: vias 20 -> 21
Changed lines of the file:
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@@
   (via (at 148.59 118.237) (size 0.6096) (drill 0.3048) (layers "F.Cu" "B.Cu") (net 2))
   (via (at 193.675 139.065) (size 0.6096) (drill 0.3048) (layers "F.Cu" "B.Cu") (net 2))
+  (via (at 164.719 135.89) (size 0.6096) (drill 0.3048) (layers "F.Cu" "B.Cu") (net 2))
   (via (at 148.59 123.317) (size 0.6096) (drill 0.3048) (layers "F.Cu" "B.Cu") (net 2))
   (via (at 148.59 119.253) (size 0.6096) (drill 0.3048) (layers "F.Cu" "B.Cu") (net 2))
@@
   (segment (start 184.658 133.65336) (end 182.19314 131.1885) (width 0.1524) (layer "B.Cu") (net 23))
   (segment (start 185.631 136.466) (end 185.431 136.466) (width 0.1524) (layer "B.Cu") (net 23))
+  (segment (start 185.631 136.466) (end 189.781 136.466) (width 0.1524) (layer "B.Cu") (net 23))
   (segment (start 184.658 135.693) (end 184.658 133.65336) (width 0.1524) (layer "B.Cu") (net 23))
   (segment (start 182.19314 131.1885) (end 177.1605 131.1885) (width 0.1524) (layer "B.Cu") (net 23))
   (segment (start 185.431 136.466) (end 184.658 135.693) (width 0.1524) (layer "B.Cu") (net 23))
+  (segment (start 185.631 132.656) (end 189.781 132.656) (width 0.1524) (layer "B.Cu") (net 24))
   (segment (start 184.091 132.656) (end 181.737 130.302) (width 0.1524) (layer "B.Cu") (net 24))
   (segment (start 185.631 132.656) (end 184.091 132.656) (width 0.1524) (layer "B.Cu") (net 24))
